Commit message: Add files via upload

File: jetnano.urdf (robot description, URDF)
Before this commit: robot jetnano, 5 links, 4 joints
Joints:
- removed joint base_link_to_odom=
- removed joint map_to_base_link=
- added joint map_to_odom=: type fixed, parent map, child odom, origin xyz=0 0 0 rpy=0 0 0
- added joint odom_to_base_link=: type fixed, parent odom, child base_link, origin xyz=0 0 0 rpy=0 0 0
- joint camera_joint: origin xyz=-0.08 0 0 rpy=0 0 -3.05 -> xyz=0 0 0 rpy=0 0 0; parent odom -> base_link
- joint laser_joint: axis 0 1 0 -> 0 0 0; origin xyz=-0.02 0 0 rpy=0 0 0 -> xyz=0 0 0 rpy=0 0 0; parent odom -> base_link

Commit message: Add files via upload

File: jetnano.urdf (robot description, URDF)
Before this commit: robot jetnano, 5 links, 4 joints
Links:
- added link world
Joints:
- added joint world_to_map=: type fixed, parent world, child map, origin xyz=0 0 0 rpy=0 0 0
- joint camera_joint: origin xyz=0 0 0 rpy=0 0 0 -> xyz=0 0 0.32 rpy=0 0 0
- joint laser_joint: origin xyz=0 0 0 rpy=0 0 0 -> xyz=0 0 0 rpy=0 0 -84.8
